Commit message: creation de ligne droite

File: data/test.urdf (robot description, URDF)
Before this commit: robot pi_robot, 3 links, 2 joints
Links:
- removed link left_wheel
- removed link right_wheel
- added link roue_droite, mass 0.1; collision cylinder length=0.02 radius=0.05; visual cylinder length=0.02 radius=0.05
- added link roue_gauche, mass 0.1; collision cylinder length=0.02 radius=0.05; visual cylinder length=0.02 radius=0.05
- added link roue_libre_arriere, mass 0.2; collision sphere radius=0.02; visual sphere radius=0.02
- added link roue_libre_avant, mass 0.2; collision sphere radius=0.02; visual sphere radius=0.02
- added link structure_horizontale, mass 0.2; visual box size=0.15 0.15 0.02
- added link structure_verticale, mass 0.2; visual box size=0.02 0.05 0.1
- link base_link: mass 2.4 -> 5; geometry visual box size=0.40 0.20 0.02
Joints:
- removed joint torso_joint_left
- removed joint torso_joint_right
- added joint joint_roue_droite: type revolute, parent base_link, child roue_droite, origin xyz=0 -0.1 0 rpy=1.57079632679 0 0, axis 0 0 1, limit lower=-3.1416 upper=3.1416 effort=10 velocity=3
- added joint joint_roue_gauche: type revolute, parent base_link, child roue_gauche, origin xyz=0 0.1 0 rpy=-1.57079632679 0 0, axis 0 0 1, limit lower=-3.1416 upper=3.1416 effort=10 velocity=3
- added joint joint_roue_libre_arriere: type fixed, parent base_link, child roue_libre_arriere, origin xyz=-0.18 0 -0.025 rpy=0 0 0
- added joint joint_roue_libre_avant: type fixed, parent base_link, child roue_libre_avant, origin xyz=0.18 0 -0.025 rpy=0 0 0
- added joint joint_structure_horizontale: type fixed, parent structure_verticale, child structure_horizontale
- added joint joint_structure_verticale: type fixed, parent base_link, child structure_verticale
